Commit message: ros systems integration

File: src/bmm3/models/BMM3/BMM3.urdf (robot description, URDF)
Before this commit: robot BMM3, 62 links, 61 joints
Joints:
- joint Wrist3Joint_left: origin xyz=0.0 0.0 0.09465 rpy=0.0 0.0 0.0 -> xyz=0.0 0.0 0.09465 rpy=0.0 -2.53 0.0
- joint Wrist3Joint_right: origin xyz=0.0 0.0 0.09465 rpy=0.0 0.0 0.0 -> xyz=0.0 0.0 0.09465 rpy=0.0 2.53 0.0
- joint connector_right: axis -1 0 0 -> (none); limit lower=0 upper=0 effort=0 velocity=0 -> (none); type revolute -> fixed
