Commit message: clean cache

File: src/robot_description/urdf/mobile_manipulator.urdf (robot description, URDF)
Before this commit: robot mobile_manipulator, 10 links, 9 joints
Links:
- added link laser_link, mass 1e-5; collision box size=0.1 0.1 0.1; visual box size=0.05 0.05 0.05
Joints:
- added joint laser_joint: type fixed, parent base_link, child laser_link, origin xyz=0.350 0 0.115 rpy=0 0 0, axis 0 1 0
